File: _saved_R2T.sch (KiCad schematic (older format))
At the start: 14 parts, among them J1 12V_Input, J2 Conn_02x01, J3 Conn_01x07, J4 Conn_01x07, J5 Conn_02x01, J6 Conn_02x01, J7 Conn_01x03, J8 Conn_01x03, U0 μA78Lxx, U1 Teensy3.5

Commit message: Added connectors still need to switch serial from x02 pin to x03 pin add ground + biger wires for cnc engraving
Parts:
- J3, J4: footprint Connector_PinSocket_2.54mm:PinSocket_1x07_P2.54mm_Vertical -> Connector_PinHeader_2.00mm:PinHeader_1x07_P2.00mm_Vertical
Changed lines of the file:
@@
 F 0 "J4" H 4850 6450 50  0000 C CNN
 F 1 "Conn_01x07" H 4850 5650 50  0000 C CNN
-F 2 "Connector_PinSocket_2.54mm:PinSocket_1x07_P2.54mm_Vertical" H 4850 6050 50  0001 C CNN
+F 2 "Connector_PinHeader_2.00mm:PinHeader_1x07_P2.00mm_Vertical" H 4850 6050 50  0001 C CNN
 F 3 "" H 4850 6050 50  0001 C CNN
 	1    4850 6050
@@
 F 0 "J3" H 4300 7200 50  0000 C CNN
 F 1 "Conn_01x07" H 4300 6400 50  0000 C CNN
-F 2 "Connector_PinSocket_2.54mm:PinSocket_1x07_P2.54mm_Vertical" H 4300 6800 50  0001 C CNN
+F 2 "Connector_PinHeader_2.00mm:PinHeader_1x07_P2.00mm_Vertical" H 4300 6800 50  0001 C CNN
 F 3 "" H 4300 6800 50  0001 C CNN
 	1    4300 6800
