File: R2T.kicad_pcb (KiCad board)
At the start: 2 copper layers, 14 parts, among them J1 12V_Input, J2 Conn_02x01, J3 Conn_01x07, J4 Conn_01x07, J5 Conn_02x01, J6 Conn_02x01, J7 Conn_01x03, J8 Conn_01x03, U0 μA78Lxx, U1 Teensy3.5

Commit message: Added a 3rd pin on the connector for the serial debug on the teensy : gnd added
Parts:
- J2: value Conn_02x01 -> Conn_01x03; footprint Connector_PinSocket_2.00mm:PinSocket_1x02_P2.00mm_Horizontal -> Connector_PinHeader_2.00mm:PinHeader_1x03_P2.00mm_Vertical
- moved J2 1.91 mm to (177.2, 35.6), turned to 180 degrees
Connections:
- U1 pad 0: Net-(J2-Pad1) -> Net-(J2-Pad2)
- U1 pad 1: Net-(J2-Pad2) -> Net-(J2-Pad1)
Routing:
- net Net-(J4-Pad3): track 10.7 -> 18.2 mm
- net Net-(J4-Pad4): track 10.8 -> 18.1 mm
- net Net-(J8-Pad1): track 18.6 -> 25.1 mm
- net Net-(J4-Pad6): track 11.3 -> 17.5 mm
- net Net-(J4-Pad5): track 11.3 -> 17.3 mm
- net Net-(J2-Pad2): track 5.30 -> 10.2 mm
- net Net-(J4-Pad7): track 11.5 -> 16.1 mm
- net Net-(J8-Pad3): track 15.0 -> 17.7 mm
- net Net-(J2-Pad1): track 5.08 -> 5.98 mm
- net GND: track 52.0 -> 52.6 mm
Other:
- net class Default: clearance 0.3 -> 0.6
- rule trace_clearance: 0.3 -> 0.6

Commit message: Finished seperating circuits on to 3 diffrent boards : teensy / ramps 0 / ramps 1. Sill need to clean and optimis for space and soder
Parts:
- removed J2, J7, J8: Conn_01x03, Connector_PinHeader_2.00mm:PinHeader_1x03_P2.00mm_Vertical
- removed J3, J4: Conn_01x07, Connector_PinHeader_2.00mm:PinHeader_1x07_P2.00mm_Vertical
- removed J5, J6: Conn_02x01, Connector_PinSocket_2.00mm:PinSocket_1x02_P2.00mm_Horizontal
- removed U0: μA78Lxx, Package_TO_SOT_SMD:SOT-223-3_TabPin2
- added Debug_Serial1: Conn_01x03, Connector_PinHeader_2.00mm:PinHeader_1x03_P2.00mm_Vertical, F.Cu at (177.3, 35.6)
- added Reg12V_5V1: μA78Lxx, Package_TO_SOT_SMD:SOT-223-3_TabPin2, F.Cu at (188.5, 19.6)
- added conn0A.b1: Conn_01x03, Connector_PinHeader_2.00mm:PinHeader_1x03_P2.00mm_Vertical, F.Cu at (149.1, 26.7)
- added conn0A.t1: Conn_01x03, Connector_PinHeader_2.00mm:PinHeader_1x03_P2.00mm_Vertical, F.Cu at (160.5, 26.7)
- added conn0B.b1: Conn_01x09, Connector_PinHeader_2.00mm:PinHeader_1x09_P2.00mm_Vertical, F.Cu at (149.1, 55.1)
- added conn0B.t1: Conn_01x09, Connector_PinHeader_2.00mm:PinHeader_1x09_P2.00mm_Vertical, F.Cu at (160.8, 55.4)
- added conn0C.b1: Conn_02x01, Connector_PinSocket_2.00mm:PinSocket_2x01_P2.00mm_Vertical, F.Cu at (149.1, 64.5)
- added conn0C.t1: Conn_02x01, Connector_PinSocket_2.00mm:PinSocket_1x02_P2.00mm_Horizontal, F.Cu at (160.8, 64.5)
- added conn0D.b1: Conn_01x07, Connector_PinHeader_2.00mm:PinHeader_1x07_P2.00mm_Vertical, F.Cu at (148.8, 68.8)
- added conn0D.t1: Conn_01x07, Connector_PinHeader_2.00mm:PinHeader_1x07_P2.00mm_Vertical, F.Cu at (161.0, 68.8)
- added conn1A.b1: conn1A.b, Connector_PinSocket_2.00mm:PinSocket_2x01_P2.00mm_Vertical, F.Cu at (211.8, 24.9)
- added conn1A.t1: conn1A.t, Connector_PinSocket_2.00mm:PinSocket_2x01_P2.00mm_Vertical, F.Cu at (208.0, 24.9)
- added conn1B.b1: Conn_01x03, Connector_PinSocket_2.00mm:PinSocket_1x03_P2.00mm_Vertical, F.Cu at (221.7, 43.9)
- added conn1B.t1: Conn_01x03, Connector_PinSocket_2.00mm:PinSocket_1x03_P2.00mm_Vertical, F.Cu at (216.7, 43.7)
- added conn1C.b1: Conn_01x13, Connector_PinSocket_2.00mm:PinSocket_1x06_P2.00mm_Vertical, F.Cu at (222.5, 94.2)
- added conn1C.t1: Conn_01x13, Connector_PinSocket_2.00mm:PinSocket_1x06_P2.00mm_Vertical, F.Cu at (216.4, 98.3)
- added conn1D.b1: Conn_01x07, Connector_PinHeader_2.00mm:PinHeader_1x07_P2.00mm_Vertical, F.Cu at (222.2, 86.4)
- added conn1D.t1: Conn_01x07, Connector_PinHeader_2.00mm:PinHeader_1x07_P2.00mm_Vertical, F.Cu at (216.4, 85.9)
- moved ARD2 15.3 mm to (228.1, 15.2)
Connections:
- U1 pad 10: Net-(ARD1-PadD26) -> Net-(U1-Pad10)
- U1 pad 11: Net-(ARD1-PadD28) -> Net-(U1-Pad11)
- U1 pad 12: Net-(ARD1-PadD24) -> Net-(U1-Pad12)
- U1 pad 2: Net-(ARD1-PadD8) -> Net-(U1-Pad2)
- U1 pad 20: Net-(ARD2-PadA14) -> Net-(U1-Pad20)
- U1 pad 21: Net-(ARD2-PadA13) -> Net-(U1-Pad21)
- U1 pad 23: Net-(ARD2-PadD10) -> Net-(U1-Pad23)
- U1 pad 27: Net-(ARD2-PadD26) -> Net-(U1-Pad27)
- U1 pad 28: Net-(ARD2-PadD28) -> Net-(U1-Pad28)
- U1 pad 29: Net-(ARD2-PadD24) -> Net-(U1-Pad29)
- U1 pad 3: Net-(ARD1-PadD9) -> Net-(U1-Pad3)
- U1 pad 30: Net-(ARD2-PadD36) -> Net-(U1-Pad30)
- U1 pad 31: Net-(ARD2-PadD34) -> Net-(U1-Pad31)
- U1 pad 32: Net-(ARD2-PadD30) -> Net-(U1-Pad32)
- U1 pad 34: Net-(ARD2-PadA2) -> Net-(U1-Pad34)
- U1 pad 35: Net-(ARD2-PadA7) -> Net-(U1-Pad35)
- U1 pad 36: Net-(ARD2-PadA6) -> Net-(U1-Pad36)
- U1 pad 37: Net-(ARD2-PadD38) -> Net-(U1-Pad37)
- U1 pad 38: Net-(ARD2-PadA1) -> Net-(U1-Pad38)
- U1 pad 39: Net-(ARD2-PadA0) -> Net-(U1-Pad39)
- U1 pad 4: Net-(ARD2-PadD8) -> Net-(U1-Pad4)
- U1 pad 5: Net-(ARD2-PadD9) -> Net-(U1-Pad5)
- U1 pad 6: Net-(ARD1-PadD10) -> Net-(U1-Pad6)
- U1 pad 7: Net-(ARD1-PadA0) -> Net-(U1-Pad7)
- U1 pad 8: Net-(ARD1-PadA1) -> Net-(U1-Pad8)
- U1 pad 9: Net-(ARD1-PadD38) -> Net-(U1-Pad9)
Routing:
- net Net-(ARD1-PadA15): track 10.3 -> 178.3 mm
- net Net-(ARD1-PadA6): track 30.9 -> 140.7 mm
- net Net-(ARD1-PadD48): track 14.0 -> 115.6 mm
- net Net-(ARD2-PadD9): track 177.9 -> 79.3 mm
- net Net-(U1-Pad19): track 16.1 -> 113.1 mm
- net Net-(ARD1-PadD36): track 44.2 -> 140.7 mm
- net Net-(ARD1-PadA7): track 31.8 -> 126.1 mm
- net Net-(ARD1-PadD46): track 14.2 -> 107.2 mm
- net Net-(U1-Pad18): track 17.5 -> 107.7 mm
- net Net-(U1-Pad17): track 17.3 -> 104.8 mm
- net Net-(ARD1-PadA13): track 14.4 -> 100.5 mm
- net Net-(ARD1-PadA14): track 15.4 -> 100.1 mm
- net Net-(U1-Pad16): track 18.1 -> 99.6 mm
- net Net-(U1-Pad14): track 10.4 -> 91.6 mm
- net Net-(ARD1-PadA8): track 5.16 -> 85.0 mm
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Other:
- net class Default: clearance 0.6 -> 0.3
- rule trace_clearance: 0.6 -> 0.3
- board text added: "Ramps 1.4 Board 0"
- board text added: "Ramps 1.4 Board 1"

Commit message: Finished cleaning
Parts:
- moved conn1A.b1 13.5 mm to (225.3, 24.9)
- moved conn0A.t1 10.9 mm to (171.4, 26.7)
- moved conn0B.t1 10.7 mm to (171.4, 55.1)
- moved conn0C.t1 10.4 mm to (171.2, 64.5)
- moved conn0D.t1 10.4 mm to (171.4, 68.8)
- moved conn1B.t1 8.40 mm to (208.3, 44.2)
- moved conn1C.t1 8.13 mm to (208.3, 98.0)
- moved conn1D.t1 8.13 mm to (208.3, 85.6)
- moved conn1C.b1 6.71 mm to (225.3, 88.1)
- moved conn1B.b1 3.57 mm to (225.3, 44.2)
- moved conn1D.b1 3.09 mm to (225.3, 85.9)
- moved C1 2.52 mm to (182.9, 18.8)
- moved C2 1.83 mm to (196.6, 18.8)
- moved conn1A.t1 0.25 mm to (208.3, 24.9)
Routing:
- net Net-(ARD1-PadA13): track 100.5 -> 192.1 mm
- net Net-(ARD1-PadA8): track 85.0 -> 166.4 mm
- net Net-(ARD1-PadD48): track 115.6 -> 168.4 mm
- net Net-(ARD1-PadD9): track 260.2 -> 242.1 mm
- net Net-(U1-Pad3.3V): track 20.2 -> 2.06 mm, vias 1 -> 0
- net Net-(ARD1-PadD8): track 244.0 -> 229.5 mm
- net Net-(ARD1-PadD10): track 250.3 -> 236.4 mm
- net Net-(ARD2-PadD9): track 79.3 -> 65.8 mm
- net Net-(ARD2-PadD8): track 79.5 -> 66.0 mm
- net Net-(ARD2-PadD10): track 62.1 -> 75.1 mm
- net Net-(ARD1-PadA15): track 178.3 -> 166.0 mm
- net Net-(U1-Pad13): track 88.2 -> 77.1 mm
- net Net-(U1-Pad2): track 22.0 -> 11.0 mm
- net Net-(U1-Pad26): track 79.0 -> 68.1 mm
- net Net-(U1-Pad22): track 52.8 -> 41.9 mm
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